Commit message: all change

File: install/my_robot_description/share/my_robot_description/urdf/m_robot.urdf (robot description, URDF)
Before this commit: robot m_robot, 8 links, 7 joints
Links:
- added link imu_link, mass 0.1
Joints:
- added joint imu_joint: type fixed, parent base_link, child imu_link, origin xyz=0 0 0.05 rpy=0 0 0
